File: Main/_autosave-Main.kicad_sch (KiCad schematic)
At the start: 16 parts, among them J1 ATMEGA, U10 TSSP58P38, U11 TSSP58P38, U12 TSSP58P38, U13 TSSP58P38, U14 TSSP58P38, U15 TSSP58P38, U2 TSSP58P38, U3 TSSP58P38, U4 TSSP58P38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

Commit message: b
Parts:
- removed U10, U11, U12, U13, U14, U15, U4, U5, U6, U7, U8, U9: TSSP58P38, OptoDevice:Vishay_MINICAST-3Pin, symbol Sensor_Proximity:TSSP58P38
Connections:
- net +3.3V: no longer U2.3 (Vs), U3.3 (Vs)
Other:
- moved on the sheet: U2
