File: dengen/dengen.kicad_sch (KiCad schematic)
At the start: 20 parts, among them J1 Conn_01x02_Pin, J2 Conn_01x02_Pin, J3 Conn_01x02_Pin, J4 Conn_01x02_Pin, J5 Conn_01x02_Pin, J6 Conn_01x02_Pin, J7 Conn_01x02_Pin, SW1 SW_DIP_x01

Commit message: Add files via upload
Parts:
- removed J3: Conn_01x02_Pin, symbol Connector:Conn_01x02_Pin
- removed R6: 2.2k, symbol Device:R
- removed R7: 3.3k, symbol Device:R
- removed SW1: SW_DIP_x01, symbol Switch:SW_DIP_x01
- removed U1: ~, symbol @toguru:toguru
- added 12V1, 3.3V2, 5V1: Conn_01x02_Pin, Connector_JST:JST_XH_B2B-XH-A_1x02_P2.50mm_Vertical, symbol Connector:Conn_01x02_Pin
- added 12V2, ON/OFF1, ON/OFF2: Conn_01x02_Pin, Connector_JST:JST_XA_S02B-XASK-1N-BN_1x02_P2.50mm_Horizontal, symbol Connector:Conn_01x02_Pin
- added C3: C, dengen:C, symbol Device:C
- added C4, C5: C, Capacitor_SMD:C_0805_2012Metric, symbol Device:C
- added R10: 680, Resistor_THT:R_Axial_DIN0207_L6.3mm_D2.5mm_P7.62mm_Horizontal, symbol Device:R
- added R12: 1.2k, Resistor_THT:R_Axial_DIN0207_L6.3mm_D2.5mm_P7.62mm_Horizontal, symbol Device:R
- added R8: 20k, Resistor_THT:R_Axial_DIN0207_L6.3mm_D2.5mm_P7.62mm_Horizontal, symbol Device:R
- added R9: 1.5k, Resistor_THT:R_Axial_DIN0207_L6.3mm_D2.5mm_P7.62mm_Horizontal, symbol Device:R
- added U1: ~, @dcdc:dcdc, symbol dcdc:dcdc
- 12V3: renamed from J2; footprint (none) -> Connector_JST:JST_XA_S02B-XASK-1N-BN_1x02_P2.50mm_Horizontal
- 3.3V1: renamed from J6; footprint (none) -> Connector_JST:JST_XH_B2B-XH-A_1x02_P2.50mm_Vertical
- 5V2: renamed from J4; footprint (none) -> Connector_JST:JST_XH_B2B-XH-A_1x02_P2.50mm_Vertical
- 5V3: renamed from J5; footprint (none) -> Connector_JST:JST_XH_B2B-XH-A_1x02_P2.50mm_Vertical
- C1, C2: footprint (none) -> Capacitor_SMD:C_0805_2012Metric
- F1: footprint (none) -> @dcdc:fuse clip
- R1, R2, R3, R4, R5: footprint (none) -> Resistor_THT:R_Axial_DIN0207_L6.3mm_D2.5mm_P7.62mm_Horizontal
- U2: footprint (none) -> @dcdc:dcdc
- Vin1: renamed from J7; footprint (none) -> Connector_JST:JST_XA_S02B-XASK-1N-BN_1x02_P2.50mm_Horizontal
- Vin2: renamed from J1; footprint (none) -> Connector_JST:JST_XA_S02B-XASK-1N-BN_1x02_P2.50mm_Horizontal
Connections:
- net +3.3V: now also 3.3V2.1 (Pin_1), C5.1, R12.1, U1.4 (Vout), U1.5 (Sense); no longer 5V3.1 (Pin_1)
- net +5V: now also 5V3.1 (Pin_1), 5V1.1 (Pin_1), C4.1, R8.1, U1.2 (Vin)
- net GND: now also 12V1.2 (Pin_2), 12V2.2 (Pin_2), 3.3V2.2 (Pin_2), 5V1.2 (Pin_2), C4.2, C5.2, R10.2, R12.2, R8.2, U1.1 (ON/Off), U1.3 (GND), U1.7 (GND)
- net VCC: now also ON/OFF1.1 (Pin_1), ON/OFF2.2 (Pin_2)
- net at F1.1, Vin1.1 (Pin_1): now also C3.1, C3.2
- net at 12V3.1 (Pin_1): now also 12V1.1 (Pin_1), 12V2.1 (Pin_1), ON/OFF1.2 (Pin_2)
- net at F1.2: now also ON/OFF2.1 (Pin_1)
- new net: R10.1, R9.2
- new net: R9.1, U1.6 (Trim)
Other:
- moved on the sheet: 12V3
